Commit message: top

File: Step1/table.urdf (robot description, URDF)
Before this commit: robot table, 6 links, 5 joints
Links:
- removed link base_link
- removed link link1
- removed link link2
- removed link link3
- removed link tool0
- added link top; visual box size=2 1 0.05
Joints:
- removed joint base_joint
- removed joint joint1
- removed joint joint2
- removed joint joint3
- removed joint tool_joint

Commit message: adding leg

File: Step1/table.urdf (robot description, URDF)
Before this commit: robot table, 2 links, 0 joints
Links:
- added link leg1; visual cylinder length=0.95 radius=0.05
Joints:
- added joint base_leg1_joint: type fixed, parent world, child leg1, origin xyz=.5 -1 0 rpy=0 0 0

Commit message: adding top link to leg1

File: Step1/table.urdf (robot description, URDF)
Before this commit: robot table, 3 links, 1 joints
Joints:
- added joint table_leg1_joint: type fixed, parent top, child leg1, origin xyz=.5 -1 0 rpy=0 0 0

Commit message: testing

File: Step1/table.urdf (robot description, URDF)
Before this commit: robot table, 3 links, 2 joints
Links:
- removed link top
Joints:
- removed joint table_leg1_joint

Commit message: fixing joint1

File: Step1/table.urdf (robot description, URDF)
Before this commit: robot table, 2 links, 1 joints
Joints:
- joint base_leg1_joint: origin xyz=.5 -1 0 rpy=0 0 0 -> xyz=0 0 .95 rpy=0 0 0

Commit message: joint fix

File: Step1/table.urdf (robot description, URDF)
Before this commit: robot table, 2 links, 1 joints
Joints:
- joint base_leg1_joint: origin xyz=0 0 .95 rpy=0 0 0 -> xyz=0 0 0 rpy=0 0 0

Commit message: fixing joint

File: Step1/table.urdf (robot description, URDF)
Before this commit: robot table, 2 links, 1 joints
Joints:
- joint base_leg1_joint: origin xyz=0 0 0 rpy=0 0 0 -> xyz=0 -1 0 rpy=0 0 0

Commit message: changing joint y

File: Step1/table.urdf (robot description, URDF)
Before this commit: robot table, 2 links, 1 joints
Joints:
- joint base_leg1_joint: origin xyz=0 -1 0 rpy=0 0 0 -> xyz=0 0 0 rpy=0 0 0

Commit message: changing a lot

File: Step1/table.urdf (robot description, URDF)
Before this commit: robot table, 2 links, 1 joints
Joints:
- joint base_leg1_joint: origin xyz=0 0 0 rpy=0 0 0 -> xyz=.5 -1 0 rpy=0 0 0

Commit message: changing joint

File: Step1/table.urdf (robot description, URDF)
Before this commit: robot table, 2 links, 1 joints
Joints:
- joint base_leg1_joint: origin xyz=.5 -1 0 rpy=0 0 0 -> xyz=.5 -1 .95 rpy=0 0 0

Commit message: changing joiong

File: Step1/table.urdf (robot description, URDF)
Before this commit: robot table, 2 links, 1 joints
Joints:
- joint base_leg1_joint: origin xyz=.5 -1 .95 rpy=0 0 0 -> xyz=.5 -1 -.95 rpy=0 0 0

Commit message: changing joing

File: Step1/table.urdf (robot description, URDF)
Before this commit: robot table, 2 links, 1 joints
Joints:
- joint base_leg1_joint: origin xyz=.5 -1 -.95 rpy=0 0 0 -> xyz=.5 -1 .95 rpy=0 0 0

Commit message: changing jiong

File: Step1/table.urdf (robot description, URDF)
Before this commit: robot table, 2 links, 1 joints
Joints:
- joint base_leg1_joint: origin xyz=.5 -1 .95 rpy=0 0 0 -> xyz=.5 -1 0 rpy=0 0 0

Commit message: adding top

File: Step1/table.urdf (robot description, URDF)
Before this commit: robot table, 2 links, 1 joints
Links:
- added link table; visual box size=1 2 0.05
Joints:
- added joint table_leg1_joint: type fixed, parent table, child leg1, origin xyz=.5 -1 0 rpy=0 0 0

Commit message: adding top

File: Step1/table.urdf (robot description, URDF)
Before this commit: robot table, 3 links, 2 joints
Links:
- removed link leg1
- removed link table
- added link top; visual box size=2 1 0.05
Joints:
- removed joint base_leg1_joint
- removed joint table_leg1_joint
- added joint top_joint: type fixed, parent world, child top_link, origin xyz=0 0 1 rpy=0 0 0

Commit message: changing names

File: Step1/table.urdf (robot description, URDF)
Before this commit: robot table, 2 links, 1 joints
Joints:
- joint top_joint: child top_link -> top

Commit message: adding leg1

File: Step1/table.urdf (robot description, URDF)
Before this commit: robot table, 2 links, 1 joints
Links:
- added link leg1; visual cylinder length=.95 radius=.05
Joints:
- added joint leg1_joint: type fixed, parent top, child leg1, origin xyz=0 0 0 rpy=0 0 0

Commit message: changing leg1

File: Step1/table.urdf (robot description, URDF)
Before this commit: robot table, 3 links, 2 joints
Joints:
- joint leg1_joint: origin xyz=0 0 0 rpy=0 0 0 -> xyz=.5 1 0 rpy=0 0 0

Commit message: fixing leg1

File: Step1/table.urdf (robot description, URDF)
Before this commit: robot table, 3 links, 2 joints
Joints:
- joint leg1_joint: origin xyz=.5 1 0 rpy=0 0 0 -> xyz=1 .5 0 rpy=0 0 0

Commit message: all links

File: Step1/table.urdf (robot description, URDF)
Before this commit: robot table, 3 links, 2 joints
Links:
- added link leg2; visual cylinder length=.95 radius=.05
- added link leg3; visual cylinder length=.95 radius=.05
- added link leg4; visual cylinder length=.95 radius=.05
Joints:
- added joint leg2_joint: type fixed, parent top, child leg2, origin xyz=1 -.5 0 rpy=0 0 0
- added joint leg3_joint: type fixed, parent top, child leg3, origin xyz=-1 -.5 0 rpy=0 0 0
- added joint leg4_joint: type fixed, parent top, child leg4, origin xyz=1 -.5 0 rpy=0 0 0

Commit message: moonshot

File: Step1/table.urdf (robot description, URDF)
Before this commit: robot table, 6 links, 5 joints
Joints:
- joint leg4_joint: origin xyz=1 -.5 0 rpy=0 0 0 -> xyz=-1 -.5 0 rpy=0 0 0

Commit message: agaian

File: Step1/table.urdf (robot description, URDF)
Before this commit: robot table, 6 links, 5 joints
Joints:
- joint leg4_joint: origin xyz=-1 -.5 0 rpy=0 0 0 -> xyz=-1 .5 0 rpy=0 0 0

Commit message: fixing frames

File: Step1/table.urdf (robot description, URDF)
Before this commit: robot table, 6 links, 5 joints
Joints:
- joint leg4_joint: origin xyz=-1 .5 0 rpy=0 0 0 -> xyz=-1.05 .45 0 rpy=0 0 0

Commit message: final (i hope)

File: Step1/table.urdf (robot description, URDF)
Before this commit: robot table, 6 links, 5 joints
Joints:
- joint leg1_joint: origin xyz=1 .5 0 rpy=0 0 0 -> xyz=.95 .45 0 rpy=0 0 0
- joint leg2_joint: origin xyz=1 -.5 0 rpy=0 0 0 -> xyz=-.95 -.45 0 rpy=0 0 0
- joint leg3_joint: origin xyz=-1 -.5 0 rpy=0 0 0 -> xyz=-.95 -.45 0 rpy=0 0 0
- joint leg4_joint: origin xyz=-1.05 .45 0 rpy=0 0 0 -> xyz=-.95 .45 0 rpy=0 0 0

Commit message: final ( i know)

File: Step1/table.urdf (robot description, URDF)
Before this commit: robot table, 6 links, 5 joints
Joints:
- joint leg3_joint: origin xyz=-.95 -.45 0 rpy=0 0 0 -> xyz=-.95 .45 0 rpy=0 0 0

Commit message: final(im sure)

File: Step1/table.urdf (robot description, URDF)
Before this commit: robot table, 6 links, 5 joints
Joints:
- joint leg3_joint: origin xyz=-.95 .45 0 rpy=0 0 0 -> xyz=.95 -.45 0 rpy=0 0 0
