Commit message: testing val

File: Step2/rrbot_macro.xacro (robot description, xacro)
@@ -5,6 +5,6 @@
     <xacro:property name="width" value="0.05" /> <!-- Square dimensions (widthxwidth) of beams -->
     <xacro:property name="height0" value="2" /> <!-- base_link -->
-    <xacro:property name="height1" value="1" /> <!-- link1 -->
-    <xacro:property name="height2" value="1" /> <!-- link2 -->
+    <xacro:property name="height1" value="2" /> <!-- link1 -->
+    <xacro:property name="height2" value="2" /> <!-- link2 -->
     <xacro:property name="axel_offset" value="0.05" /> <!-- Space between top of beam and each joint -->
     <joint name="${prefix}base_joint" type="fixed">

Commit message: idk

File: Step2/rrbot_macro.xacro (robot description, xacro)
@@ -5,6 +5,6 @@
     <xacro:property name="width" value="0.05" /> <!-- Square dimensions (widthxwidth) of beams -->
     <xacro:property name="height0" value="2" /> <!-- base_link -->
-    <xacro:property name="height1" value="2" /> <!-- link1 -->
-    <xacro:property name="height2" value="2" /> <!-- link2 -->
+    <xacro:property name="height1" value="1" /> <!-- link1 -->
+    <xacro:property name="height2" value="1" /> <!-- link2 -->
     <xacro:property name="axel_offset" value="0.05" /> <!-- Space between top of beam and each joint -->
     <joint name="${prefix}base_joint" type="fixed">
