Commit message: table top

File: Step2/table.urdf.xacro (robot description, xacro)
@@ -11,22 +11,22 @@
   </xacro:table>
   <!-- create the first leg -->
-  <xacro:leg prefix="leg1_" parent="world">
+  <!-- <xacro:leg prefix="leg1_" parent="world"> -->
     <!-- position robot in the world -->
     <origin xyz="0 0 0" rpy="0 0 0" />
-  </xacro:leg>
+  <!-- </xacro:leg> -->
   <!-- create the second leg -->
-  <xacro:table prefix="leg2_" parent="world">
+  <!-- <xacro:leg prefix="leg2_" parent="world"> -->
     <!-- position robot in the world -->
     <origin xyz="3 0 0" rpy="0 0 ${degrees(180)}" />
-  </xacro:rrbot>
+  <!-- </xacro:leg> -->
   <!-- create the third leg -->
-  <xacro:table prefix="leg3_" parent="world">
+  <!-- <xacro:leg prefix="leg3_" parent="world"> -->
     <!-- position robot in the world -->
     <origin xyz="3 0 0" rpy="0 0 ${degrees(180)}" />
-  </xacro:rrbot>
+  <!-- </xacro:leg> -->
   <!-- create the fourth leg -->
-  <xacro:table prefix="leg4_" parent="world">
+  <!-- <xacro:leg prefix="leg4_" parent="world"> -->
     <!-- position robot in the world -->
     <origin xyz="3 0 0" rpy="0 0 ${degrees(180)}" />
-  </xacro:rrbot>
+  <!-- </xacro:leg> -->
 </robot>

File: Step2/table_macro.xacro (robot description, xacro)
@@ -3,63 +3,23 @@
   <xacro:macro name="leg" params="prefix parent *origin">
     <!-- Constants for robot dimensions -->
-    <xacro:property name="width" value="0.05" /> <!-- Square dimensions (widthxwidth) of beams -->
-    <xacro:property name="height0" value="2" /> <!-- base_link -->
-    <xacro:property name="height1" value="2" /> <!-- link1 -->
-    <xacro:property name="height2" value="2" /> <!-- link2 -->
-    <xacro:property name="axel_offset" value="0.05" /> <!-- Space between top of beam and each joint -->
-    <joint name="${prefix}base_joint" type="fixed">
-      <xacro:insert_block name="origin" />
-      <parent link="${parent}" />
-      <child link="${prefix}base_link" />
-    </joint>
-    <!-- Base Link -->
-    <link name="${prefix}base_link">
-      <visual>
-        <origin xyz="0 0 ${height0/2}" rpy="0 0 0" />
-        <geometry>
-          <box size="${width} ${width} ${height0}" />
-        </geometry>
-        <material name="blue" />
-      </visual>
-    </link>
-    <joint name="${prefix}joint1" type="continuous">
-      <parent link="${prefix}base_link" />
-      <child link="${prefix}link1" />
-      <origin xyz="0 ${width} ${height0 - axel_offset}" rpy="0 0 0" />
-      <axis xyz="0 1 0" />
-    </joint>
-    <!-- Middle Link -->
-    <link name="${prefix}link1">
-      <visual>
-        <origin xyz="0 0 ${height1/2 - axel_offset}" rpy="0 0 0" />
-        <geometry>
-          <box size="${width} ${width} ${height1}" />
-        </geometry>
-        <material name="red" />
-      </visual>
-    </link>
-    <joint name="${prefix}joint2" type="continuous">
-      <parent link="${prefix}link1" />
-      <child link="${prefix}link2" />
-      <origin xyz="0 ${width} ${height1 - axel_offset*2}" rpy="0 0 0" />
-      <axis xyz="0 1 0" />
-    </joint>
-    <!-- Top Link -->
-    <link name="${prefix}link2">
-      <visual>
-        <origin xyz="0 0 ${height2/2 - axel_offset}" rpy="0 0 0" />
-        <geometry>
-          <box size="${width} ${width} ${height2}" />
-        </geometry>
-        <material name="black" />
-      </visual>
-    </link>
-    <joint name="${prefix}tool_joint" type="fixed">
-      <origin xyz="0 0 ${height2-axel_offset}" rpy="0 0 0" />
-      <parent link="${prefix}link2" />
-      <child link="${prefix}tool0" />
-    </joint>
-    <!-- Tool Link -->
-    <link name="${prefix}tool0"/>
+    <xacro:property name="table_base" value="2" /> <!-- base (x) of top -->
+    <xacro:property name="table_width" value="1" /> <!-- width (y) of top  -->
+    <xacro:property name="table_height" value=".05" /> <!-- height (z) of top -->
+  <!-- joint from "world" to "top"-->
+  <joint name="{prefix}base_joint" type="fixed">
+    <origin rpy="0 0 0" xyz="0 0 1" />
+    <parent link="${parent}" />
+    <child link="${prefix}base_link}" />
+  </joint>
+  <!-- Top Link -->
+  <link name="${prefix}base_link">
+    <visual>
+      <origin rpy="0 0 0" xyz="0 0 ${-table_height/2}" />
+      <geometry>
+        <box size="${table_base} ${table_width} ${table_height}" />
+      </geometry>
+      <material name="brown" />
+    </visual>
+  </link>
   </xacro:macro>
 </robot>

Commit message: done??

File: Step2/table.urdf.xacro (robot description, xacro)
@@ -10,23 +10,3 @@
     <origin xyz="0 0 0" rpy="0 0 0" />
   </xacro:table>
-  <!-- create the first leg -->
-  <!-- <xacro:leg prefix="leg1_" parent="world"> -->
-    <!-- position robot in the world -->
-    <origin xyz="0 0 0" rpy="0 0 0" />
-  <!-- </xacro:leg> -->
-  <!-- create the second leg -->
-  <!-- <xacro:leg prefix="leg2_" parent="world"> -->
-    <!-- position robot in the world -->
-    <origin xyz="3 0 0" rpy="0 0 ${degrees(180)}" />
-  <!-- </xacro:leg> -->
-  <!-- create the third leg -->
-  <!-- <xacro:leg prefix="leg3_" parent="world"> -->
-    <!-- position robot in the world -->
-    <origin xyz="3 0 0" rpy="0 0 ${degrees(180)}" />
-  <!-- </xacro:leg> -->
-  <!-- create the fourth leg -->
-  <!-- <xacro:leg prefix="leg4_" parent="world"> -->
-    <!-- position robot in the world -->
-    <origin xyz="3 0 0" rpy="0 0 ${degrees(180)}" />
-  <!-- </xacro:leg> -->
 </robot>

Commit message: commit

File: Step2/table.urdf.xacro (robot description, xacro)
@@ -8,5 +8,5 @@
   <xacro:table prefix="table_" parent="world">
     <!-- position robot in the world -->
-    <origin xyz="0 0 0" rpy="0 0 0" />
+    <origin xyz="0 0 1" rpy="0 0 0" />
   </xacro:table>
 </robot>
