Commit message: testing

File: Step2/table_on_rrbot.urdf.xacro (robot description, xacro)
@@ -6,5 +6,5 @@
     <link name="world" />
     <xacro:rrbot prefix="rrbot_" parent="world">
-        <origin xyz="0 0 0" rpy="0 0 0" />
+        <origin xyz="0 0 1" rpy="0 0 0" />
     </xacro:rrbot>
     <xacro:table prefix="table_" parent="rrbot_tool0">

Commit message: d

File: Step2/table_on_rrbot.urdf.xacro (robot description, xacro)
@@ -9,5 +9,5 @@
     </xacro:rrbot>
     <xacro:table prefix="table_" parent="rrbot_tool0">
-        <origin xyz="0 0 0" rpy="${pi} 0 0" />
+        <origin xyz="0 0 -1" rpy="${pi} 0 0" />
     </xacro:table>
 </robot>

Commit message: tste

File: Step2/table_on_rrbot.urdf.xacro (robot description, xacro)
@@ -6,8 +6,8 @@
     <link name="world" />
     <xacro:rrbot prefix="rrbot_" parent="world">
-        <origin xyz="0 0 0" rpy="0 0 0" />
+        <origin xyz="0 -1 0" rpy="0 0 0" />
     </xacro:rrbot>
     <xacro:table prefix="table_" parent="rrbot_tool0">
-        <origin xyz="0 0 -1" rpy="${pi} 0 0" />
+        <origin xyz="0 0 0" rpy="${pi} 0 0" />
     </xacro:table>
 </robot>

Commit message: d

File: Step2/table_on_rrbot.urdf.xacro (robot description, xacro)
@@ -9,5 +9,5 @@
     </xacro:rrbot>
     <xacro:table prefix="table_" parent="rrbot_tool0">
-        <origin xyz="0 0 0" rpy="${pi} 0 0" />
+        <origin xyz="0 0 0" rpy="${2pi} ${pi} 0" />
     </xacro:table>
 </robot>

Commit message: d

File: Step2/table_on_rrbot.urdf.xacro (robot description, xacro)
@@ -9,5 +9,5 @@
     </xacro:rrbot>
     <xacro:table prefix="table_" parent="rrbot_tool0">
-        <origin xyz="0 0 0" rpy="${2pi} ${pi} 0" />
+        <origin xyz="0 0 0" rpy="${2 * pi} ${pi} 0" />
     </xacro:table>
 </robot>
