Commit message: changing name

File: Step2/table_macro.xacro (robot description, xacro)
@@ -1,5 +1,5 @@
 <?xml version="1.0"?>
 <robot xmlns:xacro="http://www.ros.org/wiki/xacro">
-  <xacro:macro name="leg" params="prefix parent *origin">
+  <xacro:macro name="table" params="prefix parent *origin">
     <!-- Constants for robot dimensions -->
     <xacro:property name="table_base" value="2" /> <!-- base (x) of top -->

Commit message: fixing prefixs

File: Step2/table_macro.xacro (robot description, xacro)
@@ -3,10 +3,11 @@
   <xacro:macro name="table" params="prefix parent *origin">
     <!-- Constants for robot dimensions -->
-    <xacro:property name="table_base" value="2" /> <!-- base (x) of top -->
+    <xacro:property name="table_length" value="2" /> <!-- base (x) of top -->
     <xacro:property name="table_width" value="1" /> <!-- width (y) of top  -->
-    <xacro:property name="table_height" value=".05" /> <!-- height (z) of top -->
+    <xacro:property name="table_height" value="1" /> <!-- height (z) of top -->
+    <xacro:property name="table_thickness" value=".05" /> <!-- height (z) of top -->
   <!-- joint from "world" to "top"-->
-  <joint name="{prefix}base_joint" type="fixed">
-    <origin rpy="0 0 0" xyz="0 0 1" />
+  <joint name="${prefix}base_joint" type="fixed">
+    <origin rpy="0 0 0" xyz="0 0 ${table_height}" />
     <parent link="${parent}" />
     <child link="${prefix}base_link}" />
@@ -15,7 +16,7 @@
   <link name="${prefix}base_link">
     <visual>
-      <origin rpy="0 0 0" xyz="0 0 ${-table_height/2}" />
+      <origin rpy="0 0 0" xyz="0 0 ${-table_thickness/2}" />
       <geometry>
-        <box size="${table_base} ${table_width} ${table_height}" />
+        <box size="${table_base} ${table_width} ${table_thickness}" />
       </geometry>
       <material name="brown" />

Commit message: fixing length

File: Step2/table_macro.xacro (robot description, xacro)
@@ -18,5 +18,5 @@
       <origin rpy="0 0 0" xyz="0 0 ${-table_thickness/2}" />
       <geometry>
-        <box size="${table_base} ${table_width} ${table_thickness}" />
+        <box size="${table_length} ${table_width} ${table_thickness}" />
       </geometry>
       <material name="brown" />

Commit message: syntax error

File: Step2/table_macro.xacro (robot description, xacro)
@@ -11,5 +11,5 @@
     <origin rpy="0 0 0" xyz="0 0 ${table_height}" />
     <parent link="${parent}" />
-    <child link="${prefix}base_link}" />
+    <child link="${prefix}base_link" />
   </joint>
   <!-- Top Link -->

Commit message: done?

File: Step2/table_macro.xacro (robot description, xacro)
@@ -7,4 +7,6 @@
     <xacro:property name="table_height" value="1" /> <!-- height (z) of top -->
     <xacro:property name="table_thickness" value=".05" /> <!-- height (z) of top -->
+    <xacro:property name="leg_length" value="${table_height - table_thickness}" /> <!-- height leg -->
+    <xacro:property name="leg_radius" value="0.05" /> <!-- radius of leg -->
   <!-- joint from "world" to "top"-->
   <joint name="${prefix}base_joint" type="fixed">
@@ -23,4 +25,68 @@
     </visual>
   </link>
+  <!-- joint from "top" to "Leg1"-->
+  <joint name="${prefix}leg1_joint" type="fixed">
+    <origin rpy="0 0 0" xyz="${leg_length} ${table_height - (2 * table_thickness) / 2)} 0" />
+    <parent link="{prefix}base_link" />
+    <child link="{prefix}leg1" />
+  </joint>
+  <!-- Leg1 Link -->
+  <link name="${prefix}leg1">
+    <visual>
+      <origin rpy="0 0 0" xyz="0 0 ${-(table_height + table_thickness) / 2}" />
+      <geometry>
+        <cylinder radius="${leg_radius}" length="${leg_length}" />
+      </geometry>
+      <material name="light_grey" />
+    </visual>
+  </link>
+  <!-- joint from "top" to "Leg2"-->
+  <joint name="${prefix}leg2_joint" type="fixed">
+    <origin rpy="0 0 0" xyz="${-leg_length} ${table_height - (2 * table_thickness) / 2)} 0" />
+    <parent link="{prefix}base_link" />
+    <child link="{prefix}leg2" />
+  </joint>
+  <!-- Leg2 Link -->
+  <link name="${prefix}leg_link_2">
+    <visual>
+      <origin rpy="0 0 0" xyz="0 0 ${-(table_height + table_thickness) / 2}" />
+      <geometry>
+        <cylinder radius="${leg_radius}" length="${leg_length}" />
+      </geometry>
+      <material name="light_grey" />
+    </visual>
+  </link>
+  <!-- joint from "top" to "leg3"-->
+  <joint name="${prefix}leg3_joint" type="fixed">
+    <origin rpy="0 0 0" xyz="${leg_length} -${table_height - (2 * table_thickness) / 2)} 0" />
+    <parent link="{prefix}base_link" />
+    <child link="{prefix}leg_link_3" />
+  </joint>
+  <!-- Leg3 Link -->
+  <link name="${prefix}leg_link_3">
+    <visual>
+      <origin rpy="0 0 0" xyz="0 0 -${(table_height + table_thickness) / 2}" />
+      <geometry>
+        <cylinder radius="${leg_radius}" length="${leg_length}" />
+      </geometry>
+      <material name="light_grey" />
+    </visual>
+  </link>
+  <!-- joint from "top" to "leg4"-->
+  <joint name="${prefix}leg4_joint" type="fixed">
+    <origin rpy="0 0 0" xyz="-${leg_length} -${table_height - (2 * table_thickness) / 2)} 0" />
+    <parent link="{prefix}base_link" />
+    <child link="{prefix}leg_link_4" />
+  </joint>
+  <!-- Leg4 Link -->
+  <link name="${prefix}leg_link_4">
+    <visual>
+      <origin rpy="0 0 0" xyz="0 0 -${(table_height + table_thickness) / 2}" />
+      <geometry>
+        <cylinder radius="${leg_radius}" length="${leg_length}" />
+      </geometry>
+      <material name="light_grey" />
+    </visual>
+  </link>
   </xacro:macro>
 </robot>

Commit message: fixing parenthesis

File: Step2/table_macro.xacro (robot description, xacro)
@@ -27,5 +27,5 @@
   <!-- joint from "top" to "Leg1"-->
   <joint name="${prefix}leg1_joint" type="fixed">
-    <origin rpy="0 0 0" xyz="${leg_length} ${table_height - (2 * table_thickness) / 2)} 0" />
+    <origin rpy="0 0 0" xyz="${leg_length} ${(table_height - (2 * table_thickness) / 2)} 0" />
     <parent link="{prefix}base_link" />
     <child link="{prefix}leg1" />
@@ -43,5 +43,5 @@
   <!-- joint from "top" to "Leg2"-->
   <joint name="${prefix}leg2_joint" type="fixed">
-    <origin rpy="0 0 0" xyz="${-leg_length} ${table_height - (2 * table_thickness) / 2)} 0" />
+    <origin rpy="0 0 0" xyz="${-leg_length} ${(table_height - (2 * table_thickness) / 2)} 0" />
     <parent link="{prefix}base_link" />
     <child link="{prefix}leg2" />
@@ -59,5 +59,5 @@
   <!-- joint from "top" to "leg3"-->
   <joint name="${prefix}leg3_joint" type="fixed">
-    <origin rpy="0 0 0" xyz="${leg_length} -${table_height - (2 * table_thickness) / 2)} 0" />
+    <origin rpy="0 0 0" xyz="${leg_length} -${(table_height - (2 * table_thickness) / 2)} 0" />
     <parent link="{prefix}base_link" />
     <child link="{prefix}leg_link_3" />
@@ -75,5 +75,5 @@
   <!-- joint from "top" to "leg4"-->
   <joint name="${prefix}leg4_joint" type="fixed">
-    <origin rpy="0 0 0" xyz="-${leg_length} -${table_height - (2 * table_thickness) / 2)} 0" />
+    <origin rpy="0 0 0" xyz="-${leg_length} -${(table_height - (2 * table_thickness) / 2)} 0" />
     <parent link="{prefix}base_link" />
     <child link="{prefix}leg_link_4" />

Commit message: testing leg1

File: Step2/table_macro.xacro (robot description, xacro)
@@ -41,5 +41,5 @@
     </visual>
   </link>
-  <!-- joint from "top" to "Leg2"-->
+  <!-- joint from "top" to "Leg2"
   <joint name="${prefix}leg2_joint" type="fixed">
     <origin rpy="0 0 0" xyz="${-leg_length} ${(table_height - (2 * table_thickness) / 2)} 0" />
@@ -88,5 +88,5 @@
       <material name="light_grey" />
     </visual>
-  </link>
+  </link> -->
   </xacro:macro>
 </robot>

Commit message: comments

File: Step2/table_macro.xacro (robot description, xacro)
@@ -41,12 +41,12 @@
     </visual>
   </link>
-  <!-- joint from "top" to "Leg2"
-  <joint name="${prefix}leg2_joint" type="fixed">
+  <!--joint from "top" to "Leg2"-->
+  <!-- <joint name="${prefix}leg2_joint" type="fixed"> -->
     <origin rpy="0 0 0" xyz="${-leg_length} ${(table_height - (2 * table_thickness) / 2)} 0" />
     <parent link="{prefix}base_link" />
     <child link="{prefix}leg2" />
-  </joint>
+  <!-- </joint> -->
   <!-- Leg2 Link -->
-  <link name="${prefix}leg_link_2">
+  <!-- <link name="${prefix}leg_link_2"> -->
     <visual>
       <origin rpy="0 0 0" xyz="0 0 ${-(table_height + table_thickness) / 2}" />
@@ -56,13 +56,13 @@
       <material name="light_grey" />
     </visual>
-  </link>
+  <!-- </link> -->
   <!-- joint from "top" to "leg3"-->
-  <joint name="${prefix}leg3_joint" type="fixed">
+  <!-- <joint name="${prefix}leg3_joint" type="fixed"> -->
     <origin rpy="0 0 0" xyz="${leg_length} -${(table_height - (2 * table_thickness) / 2)} 0" />
     <parent link="{prefix}base_link" />
     <child link="{prefix}leg_link_3" />
-  </joint>
+  <!-- </joint> -->
   <!-- Leg3 Link -->
-  <link name="${prefix}leg_link_3">
+  <!-- <link name="${prefix}leg_link_3"> -->
     <visual>
       <origin rpy="0 0 0" xyz="0 0 -${(table_height + table_thickness) / 2}" />
@@ -72,13 +72,13 @@
       <material name="light_grey" />
     </visual>
-  </link>
+  <!-- </link> -->
   <!-- joint from "top" to "leg4"-->
-  <joint name="${prefix}leg4_joint" type="fixed">
+  <!-- <joint name="${prefix}leg4_joint" type="fixed"> -->
     <origin rpy="0 0 0" xyz="-${leg_length} -${(table_height - (2 * table_thickness) / 2)} 0" />
     <parent link="{prefix}base_link" />
     <child link="{prefix}leg_link_4" />
-  </joint>
+  <!-- </joint> -->
   <!-- Leg4 Link -->
-  <link name="${prefix}leg_link_4">
+  <!-- <link name="${prefix}leg_link_4"> -->
     <visual>
       <origin rpy="0 0 0" xyz="0 0 -${(table_height + table_thickness) / 2}" />
@@ -88,5 +88,5 @@
       <material name="light_grey" />
     </visual>
-  </link> -->
+  <!-- </link> -->
   </xacro:macro>
 </robot>

Commit message: final?

File: Step2/table_macro.xacro (robot description, xacro)
@@ -28,6 +28,6 @@
   <joint name="${prefix}leg1_joint" type="fixed">
     <origin rpy="0 0 0" xyz="${leg_length} ${(table_height - (2 * table_thickness) / 2)} 0" />
-    <parent link="{prefix}base_link" />
-    <child link="{prefix}leg1" />
+    <parent link="${prefix}base_link" />
+    <child link="${prefix}leg1" />
   </joint>
   <!-- Leg1 Link -->
@@ -42,11 +42,11 @@
   </link>
   <!--joint from "top" to "Leg2"-->
-  <!-- <joint name="${prefix}leg2_joint" type="fixed"> -->
+  <joint name="${prefix}leg2_joint" type="fixed">
     <origin rpy="0 0 0" xyz="${-leg_length} ${(table_height - (2 * table_thickness) / 2)} 0" />
-    <parent link="{prefix}base_link" />
-    <child link="{prefix}leg2" />
-  <!-- </joint> -->
+    <parent link="${prefix}base_link" />
+    <child link="${prefix}leg2" />
+  </joint>
   <!-- Leg2 Link -->
-  <!-- <link name="${prefix}leg_link_2"> -->
+  <link name="${prefix}leg_link_2">
     <visual>
       <origin rpy="0 0 0" xyz="0 0 ${-(table_height + table_thickness) / 2}" />
@@ -56,13 +56,13 @@
       <material name="light_grey" />
     </visual>
-  <!-- </link> -->
+  </link>
   <!-- joint from "top" to "leg3"-->
-  <!-- <joint name="${prefix}leg3_joint" type="fixed"> -->
+  <joint name="${prefix}leg3_joint" type="fixed">
     <origin rpy="0 0 0" xyz="${leg_length} -${(table_height - (2 * table_thickness) / 2)} 0" />
-    <parent link="{prefix}base_link" />
-    <child link="{prefix}leg_link_3" />
-  <!-- </joint> -->
+    <parent link="${prefix}base_link" />
+    <child link="${prefix}leg_link_3" />
+  </joint>
   <!-- Leg3 Link -->
-  <!-- <link name="${prefix}leg_link_3"> -->
+  <link name="${prefix}leg_link_3">
     <visual>
       <origin rpy="0 0 0" xyz="0 0 -${(table_height + table_thickness) / 2}" />
@@ -72,13 +72,13 @@
       <material name="light_grey" />
     </visual>
-  <!-- </link> -->
+  </link>
   <!-- joint from "top" to "leg4"-->
-  <!-- <joint name="${prefix}leg4_joint" type="fixed"> -->
+  <joint name="${prefix}leg4_joint" type="fixed">
     <origin rpy="0 0 0" xyz="-${leg_length} -${(table_height - (2 * table_thickness) / 2)} 0" />
-    <parent link="{prefix}base_link" />
-    <child link="{prefix}leg_link_4" />
-  <!-- </joint> -->
+    <parent link="${prefix}base_link" />
+    <child link="${prefix}leg_link_4" />
+  </joint>
   <!-- Leg4 Link -->
-  <!-- <link name="${prefix}leg_link_4"> -->
+  <link name="${prefix}leg_link_4">
     <visual>
       <origin rpy="0 0 0" xyz="0 0 -${(table_height + table_thickness) / 2}" />
@@ -88,5 +88,5 @@
       <material name="light_grey" />
     </visual>
-  <!-- </link> -->
+  </link>
   </xacro:macro>
 </robot>

Commit message: finallll

File: Step2/table_macro.xacro (robot description, xacro)
@@ -45,5 +45,5 @@
     <origin rpy="0 0 0" xyz="${-leg_length} ${(table_height - (2 * table_thickness) / 2)} 0" />
     <parent link="${prefix}base_link" />
-    <child link="${prefix}leg2" />
+    <child link="${prefix}leg_link_2" />
   </joint>
   <!-- Leg2 Link -->

Commit message: fixing positions

File: Step2/table_macro.xacro (robot description, xacro)
@@ -27,5 +27,5 @@
   <!-- joint from "top" to "Leg1"-->
   <joint name="${prefix}leg1_joint" type="fixed">
-    <origin rpy="0 0 0" xyz="${leg_length} ${(table_height - (2 * table_thickness) / 2)} 0" />
+    <origin rpy="0 0 0" xyz="${leg_length} ${(table_width / 2) - leg_radius} 0" />
     <parent link="${prefix}base_link" />
     <child link="${prefix}leg1" />
@@ -43,5 +43,5 @@
   <!--joint from "top" to "Leg2"-->
   <joint name="${prefix}leg2_joint" type="fixed">
-    <origin rpy="0 0 0" xyz="${-leg_length} ${(table_height - (2 * table_thickness) / 2)} 0" />
+    <origin rpy="0 0 0" xyz="${-leg_length} ${(table_width / 2) - leg_radius} 0" />
     <parent link="${prefix}base_link" />
     <child link="${prefix}leg_link_2" />
@@ -59,5 +59,5 @@
   <!-- joint from "top" to "leg3"-->
   <joint name="${prefix}leg3_joint" type="fixed">
-    <origin rpy="0 0 0" xyz="${leg_length} -${(table_height - (2 * table_thickness) / 2)} 0" />
+    <origin rpy="0 0 0" xyz="${leg_length} -${(table_width / 2) - leg_radius} 0" />
     <parent link="${prefix}base_link" />
     <child link="${prefix}leg_link_3" />
@@ -75,5 +75,5 @@
   <!-- joint from "top" to "leg4"-->
   <joint name="${prefix}leg4_joint" type="fixed">
-    <origin rpy="0 0 0" xyz="-${leg_length} -${(table_height - (2 * table_thickness) / 2)} 0" />
+    <origin rpy="0 0 0" xyz="-${leg_length} -${(table_width / 2) - leg_radius} 0" />
     <parent link="${prefix}base_link" />
     <child link="${prefix}leg_link_4" />

Commit message: new vals

File: Step2/table_macro.xacro (robot description, xacro)
@@ -3,6 +3,6 @@
   <xacro:macro name="table" params="prefix parent *origin">
     <!-- Constants for robot dimensions -->
-    <xacro:property name="table_length" value="2" /> <!-- base (x) of top -->
-    <xacro:property name="table_width" value="1" /> <!-- width (y) of top  -->
+    <xacro:property name="table_length" value="5" /> <!-- base (x) of top -->
+    <xacro:property name="table_width" value="2" /> <!-- width (y) of top  -->
     <xacro:property name="table_height" value="1" /> <!-- height (z) of top -->
     <xacro:property name="table_thickness" value=".05" /> <!-- height (z) of top -->

Commit message: fubak

File: Step2/table_macro.xacro (robot description, xacro)
@@ -27,5 +27,5 @@
   <!-- joint from "top" to "Leg1"-->
   <joint name="${prefix}leg1_joint" type="fixed">
-    <origin rpy="0 0 0" xyz="${leg_length} ${(table_width / 2) - leg_radius} 0" />
+    <origin rpy="0 0 0" xyz="${(leg_length / 2) - leg_radius} ${(table_width / 2) - leg_radius} 0" />
     <parent link="${prefix}base_link" />
     <child link="${prefix}leg1" />
@@ -43,5 +43,5 @@
   <!--joint from "top" to "Leg2"-->
   <joint name="${prefix}leg2_joint" type="fixed">
-    <origin rpy="0 0 0" xyz="${-leg_length} ${(table_width / 2) - leg_radius} 0" />
+    <origin rpy="0 0 0" xyz="${(leg_length / 2) - leg_radius} ${-leg_length} ${(table_width / 2) - leg_radius} 0" />
     <parent link="${prefix}base_link" />
     <child link="${prefix}leg_link_2" />
@@ -59,5 +59,5 @@
   <!-- joint from "top" to "leg3"-->
   <joint name="${prefix}leg3_joint" type="fixed">
-    <origin rpy="0 0 0" xyz="${leg_length} -${(table_width / 2) - leg_radius} 0" />
+    <origin rpy="0 0 0" xyz="${(leg_length / 2) - leg_radius} ${leg_length} -${(table_width / 2) - leg_radius} 0" />
     <parent link="${prefix}base_link" />
     <child link="${prefix}leg_link_3" />
@@ -75,5 +75,5 @@
   <!-- joint from "top" to "leg4"-->
   <joint name="${prefix}leg4_joint" type="fixed">
-    <origin rpy="0 0 0" xyz="-${leg_length} -${(table_width / 2) - leg_radius} 0" />
+    <origin rpy="0 0 0" xyz="${(leg_length / 2) - leg_radius} -${leg_length} -${(table_width / 2) - leg_radius} 0" />
     <parent link="${prefix}base_link" />
     <child link="${prefix}leg_link_4" />

Commit message: ugh

File: Step2/table_macro.xacro (robot description, xacro)
@@ -27,5 +27,5 @@
   <!-- joint from "top" to "Leg1"-->
   <joint name="${prefix}leg1_joint" type="fixed">
-    <origin rpy="0 0 0" xyz="${(leg_length / 2) - leg_radius} ${(table_width / 2) - leg_radius} 0" />
+    <origin rpy="0 0 0" xyz="-${(leg_length / 2) - leg_radius} ${(table_width / 2) - leg_radius} 0" />
     <parent link="${prefix}base_link" />
     <child link="${prefix}leg1" />
@@ -43,5 +43,5 @@
   <!--joint from "top" to "Leg2"-->
   <joint name="${prefix}leg2_joint" type="fixed">
-    <origin rpy="0 0 0" xyz="${(leg_length / 2) - leg_radius} ${-leg_length} ${(table_width / 2) - leg_radius} 0" />
+    <origin rpy="0 0 0" xyz="-${(leg_length / 2) - leg_radius}  ${(table_width / 2) - leg_radius} 0" />
     <parent link="${prefix}base_link" />
     <child link="${prefix}leg_link_2" />
@@ -59,5 +59,5 @@
   <!-- joint from "top" to "leg3"-->
   <joint name="${prefix}leg3_joint" type="fixed">
-    <origin rpy="0 0 0" xyz="${(leg_length / 2) - leg_radius} ${leg_length} -${(table_width / 2) - leg_radius} 0" />
+    <origin rpy="0 0 0" xyz="${(leg_length / 2) - leg_radius} -${(table_width / 2) - leg_radius} 0" />
     <parent link="${prefix}base_link" />
     <child link="${prefix}leg_link_3" />
@@ -75,5 +75,5 @@
   <!-- joint from "top" to "leg4"-->
   <joint name="${prefix}leg4_joint" type="fixed">
-    <origin rpy="0 0 0" xyz="${(leg_length / 2) - leg_radius} -${leg_length} -${(table_width / 2) - leg_radius} 0" />
+    <origin rpy="0 0 0" xyz="-${(leg_length / 2) - leg_radius} -${(table_width / 2) - leg_radius} 0" />
     <parent link="${prefix}base_link" />
     <child link="${prefix}leg_link_4" />

Commit message: final

File: Step2/table_macro.xacro (robot description, xacro)
@@ -27,5 +27,5 @@
   <!-- joint from "top" to "Leg1"-->
   <joint name="${prefix}leg1_joint" type="fixed">
-    <origin rpy="0 0 0" xyz="-${(leg_length / 2) - leg_radius} ${(table_width / 2) - leg_radius} 0" />
+    <origin rpy="0 0 0" xyz="${(leg_length) - leg_radius} ${(table_width / 2) - leg_radius} 0" />
     <parent link="${prefix}base_link" />
     <child link="${prefix}leg1" />
@@ -43,5 +43,5 @@
   <!--joint from "top" to "Leg2"-->
   <joint name="${prefix}leg2_joint" type="fixed">
-    <origin rpy="0 0 0" xyz="-${(leg_length / 2) - leg_radius}  ${(table_width / 2) - leg_radius} 0" />
+    <origin rpy="0 0 0" xyz="-${(leg_length) - leg_radius}  ${(table_width / 2) - leg_radius} 0" />
     <parent link="${prefix}base_link" />
     <child link="${prefix}leg_link_2" />
@@ -59,5 +59,5 @@
   <!-- joint from "top" to "leg3"-->
   <joint name="${prefix}leg3_joint" type="fixed">
-    <origin rpy="0 0 0" xyz="${(leg_length / 2) - leg_radius} -${(table_width / 2) - leg_radius} 0" />
+    <origin rpy="0 0 0" xyz="${(leg_length) - leg_radius} -${(table_width / 2) - leg_radius} 0" />
     <parent link="${prefix}base_link" />
     <child link="${prefix}leg_link_3" />
@@ -75,5 +75,5 @@
   <!-- joint from "top" to "leg4"-->
   <joint name="${prefix}leg4_joint" type="fixed">
-    <origin rpy="0 0 0" xyz="-${(leg_length / 2) - leg_radius} -${(table_width / 2) - leg_radius} 0" />
+    <origin rpy="0 0 0" xyz="-${(leg_length) - leg_radius} -${(table_width / 2) - leg_radius} 0" />
     <parent link="${prefix}base_link" />
     <child link="${prefix}leg_link_4" />

Commit message: ugh

File: Step2/table_macro.xacro (robot description, xacro)
@@ -27,5 +27,5 @@
   <!-- joint from "top" to "Leg1"-->
   <joint name="${prefix}leg1_joint" type="fixed">
-    <origin rpy="0 0 0" xyz="${(leg_length) - leg_radius} ${(table_width / 2) - leg_radius} 0" />
+    <origin rpy="0 0 0" xyz="${(table_length) - leg_radius} ${(table_width / 2) - leg_radius} 0" />
     <parent link="${prefix}base_link" />
     <child link="${prefix}leg1" />
@@ -43,5 +43,5 @@
   <!--joint from "top" to "Leg2"-->
   <joint name="${prefix}leg2_joint" type="fixed">
-    <origin rpy="0 0 0" xyz="-${(leg_length) - leg_radius}  ${(table_width / 2) - leg_radius} 0" />
+    <origin rpy="0 0 0" xyz="-${(table_length) - leg_radius}  ${(table_width / 2) - leg_radius} 0" />
     <parent link="${prefix}base_link" />
     <child link="${prefix}leg_link_2" />
@@ -59,5 +59,5 @@
   <!-- joint from "top" to "leg3"-->
   <joint name="${prefix}leg3_joint" type="fixed">
-    <origin rpy="0 0 0" xyz="${(leg_length) - leg_radius} -${(table_width / 2) - leg_radius} 0" />
+    <origin rpy="0 0 0" xyz="${(table_length) - leg_radius} -${(table_width / 2) - leg_radius} 0" />
     <parent link="${prefix}base_link" />
     <child link="${prefix}leg_link_3" />
@@ -75,5 +75,5 @@
   <!-- joint from "top" to "leg4"-->
   <joint name="${prefix}leg4_joint" type="fixed">
-    <origin rpy="0 0 0" xyz="-${(leg_length) - leg_radius} -${(table_width / 2) - leg_radius} 0" />
+    <origin rpy="0 0 0" xyz="-${(table_length) - leg_radius} -${(table_width / 2) - leg_radius} 0" />
     <parent link="${prefix}base_link" />
     <child link="${prefix}leg_link_4" />
