Commit message: finally

File: Step2/table_macro.xacro (robot description, xacro)
@@ -27,5 +27,5 @@
   <!-- joint from "top" to "Leg1"-->
   <joint name="${prefix}leg1_joint" type="fixed">
-    <origin rpy="0 0 0" xyz="${(table_length) - leg_radius} ${(table_width / 2) - leg_radius} 0" />
+    <origin rpy="0 0 0" xyz="${(table_length /2) - leg_radius} ${(table_width / 2) - leg_radius} 0" />
     <parent link="${prefix}base_link" />
     <child link="${prefix}leg1" />
@@ -43,5 +43,5 @@
   <!--joint from "top" to "Leg2"-->
   <joint name="${prefix}leg2_joint" type="fixed">
-    <origin rpy="0 0 0" xyz="-${(table_length) - leg_radius}  ${(table_width / 2) - leg_radius} 0" />
+    <origin rpy="0 0 0" xyz="-${(table_length /2) - leg_radius}  ${(table_width / 2) - leg_radius} 0" />
     <parent link="${prefix}base_link" />
     <child link="${prefix}leg_link_2" />
@@ -59,5 +59,5 @@
   <!-- joint from "top" to "leg3"-->
   <joint name="${prefix}leg3_joint" type="fixed">
-    <origin rpy="0 0 0" xyz="${(table_length) - leg_radius} -${(table_width / 2) - leg_radius} 0" />
+    <origin rpy="0 0 0" xyz="${(table_length / 2) - leg_radius} -${(table_width / 2) - leg_radius} 0" />
     <parent link="${prefix}base_link" />
     <child link="${prefix}leg_link_3" />
@@ -75,5 +75,5 @@
   <!-- joint from "top" to "leg4"-->
   <joint name="${prefix}leg4_joint" type="fixed">
-    <origin rpy="0 0 0" xyz="-${(table_length) - leg_radius} -${(table_width / 2) - leg_radius} 0" />
+    <origin rpy="0 0 0" xyz="-${(table_length /2) - leg_radius} -${(table_width / 2) - leg_radius} 0" />
     <parent link="${prefix}base_link" />
     <child link="${prefix}leg_link_4" />

Commit message: idk maybe

File: Step2/table_macro.xacro (robot description, xacro)
@@ -10,5 +10,5 @@
     <xacro:property name="leg_radius" value="0.05" /> <!-- radius of leg -->
   <!-- joint from "world" to "top"-->
-  <joint name="${prefix}base_joint" type="fixed">
+  <joint name="table_top" type="fixed">
     <origin rpy="0 0 0" xyz="0 0 ${table_height}" />
     <parent link="${parent}" />

Commit message: uhh

File: Step2/table_macro.xacro (robot description, xacro)
@@ -10,11 +10,11 @@
     <xacro:property name="leg_radius" value="0.05" /> <!-- radius of leg -->
   <!-- joint from "world" to "top"-->
-  <joint name="table_top" type="fixed">
+  <joint name="table_world_joint" type="fixed">
     <origin rpy="0 0 0" xyz="0 0 ${table_height}" />
     <parent link="${parent}" />
-    <child link="${prefix}base_link" />
+    <child link="table_top" />
   </joint>
   <!-- Top Link -->
-  <link name="${prefix}base_link">
+  <link name="table_top">
     <visual>
       <origin rpy="0 0 0" xyz="0 0 ${-table_thickness/2}" />

Commit message: hmm

File: Step2/table_macro.xacro (robot description, xacro)
@@ -10,5 +10,5 @@
     <xacro:property name="leg_radius" value="0.05" /> <!-- radius of leg -->
   <!-- joint from "world" to "top"-->
-  <joint name="table_world_joint" type="fixed">
+  <joint name="table_base_joint" type="fixed">
     <origin rpy="0 0 0" xyz="0 0 ${table_height}" />
     <parent link="${parent}" />
@@ -28,5 +28,5 @@
   <joint name="${prefix}leg1_joint" type="fixed">
     <origin rpy="0 0 0" xyz="${(table_length /2) - leg_radius} ${(table_width / 2) - leg_radius} 0" />
-    <parent link="${prefix}base_link" />
+    <parent link="table_top" />
     <child link="${prefix}leg1" />
   </joint>
@@ -44,5 +44,5 @@
   <joint name="${prefix}leg2_joint" type="fixed">
     <origin rpy="0 0 0" xyz="-${(table_length /2) - leg_radius}  ${(table_width / 2) - leg_radius} 0" />
-    <parent link="${prefix}base_link" />
+    <parent link="table_top" />
     <child link="${prefix}leg_link_2" />
   </joint>
@@ -60,5 +60,5 @@
   <joint name="${prefix}leg3_joint" type="fixed">
     <origin rpy="0 0 0" xyz="${(table_length / 2) - leg_radius} -${(table_width / 2) - leg_radius} 0" />
-    <parent link="${prefix}base_link" />
+    <parent link="table_top" />
     <child link="${prefix}leg_link_3" />
   </joint>
@@ -76,5 +76,5 @@
   <joint name="${prefix}leg4_joint" type="fixed">
     <origin rpy="0 0 0" xyz="-${(table_length /2) - leg_radius} -${(table_width / 2) - leg_radius} 0" />
-    <parent link="${prefix}base_link" />
+    <parent link="table_top" />
     <child link="${prefix}leg_link_4" />
   </joint>

Commit message: ik

File: Step2/table_macro.xacro (robot description, xacro)
@@ -11,5 +11,5 @@
   <!-- joint from "world" to "top"-->
   <joint name="table_base_joint" type="fixed">
-    <origin rpy="0 0 0" xyz="0 0 ${table_height}" />
+    <origin rpy="0 0 1" xyz="0 0 ${table_height}" />
     <parent link="${parent}" />
     <child link="table_top" />

File: Step2/table_on_rrbot.urdf.xacro (robot description, xacro)
@@ -6,5 +6,5 @@
     <link name="world" />
     <xacro:rrbot prefix="rrbot_" parent="world">
-        <origin xyz="0 0 1" rpy="0 0 0" />
+        <origin xyz="0 0 0" rpy="0 0 0" />
     </xacro:rrbot>
     <xacro:table prefix="table_" parent="rrbot_tool0">

Commit message: oops

File: Step2/table_macro.xacro (robot description, xacro)
@@ -11,5 +11,5 @@
   <!-- joint from "world" to "top"-->
   <joint name="table_base_joint" type="fixed">
-    <origin rpy="0 0 1" xyz="0 0 ${table_height}" />
+    <origin rpy="0 0 0" xyz="0 0 ${table_height}" />
     <parent link="${parent}" />
     <child link="table_top" />

Commit message: k

File: Step2/table_macro.xacro (robot description, xacro)
@@ -11,5 +11,5 @@
   <!-- joint from "world" to "top"-->
   <joint name="table_base_joint" type="fixed">
-    <origin rpy="0 0 0" xyz="0 0 ${table_height}" />
+    <origin rpy="0 0 0" xyz="0 0 0" />
     <parent link="${parent}" />
     <child link="table_top" />

File: Step2/table_on_rrbot.urdf.xacro (robot description, xacro)
@@ -6,5 +6,5 @@
     <link name="world" />
     <xacro:rrbot prefix="rrbot_" parent="world">
-        <origin xyz="0 -1 0" rpy="0 0 0" />
+        <origin xyz="0 0 0" rpy="0 0 0" />
     </xacro:rrbot>
     <xacro:table prefix="table_" parent="rrbot_tool0">

Commit message: ifk

File: Step2/table_macro.xacro (robot description, xacro)
@@ -18,5 +18,5 @@
   <link name="table_top">
     <visual>
-      <origin rpy="0 0 0" xyz="0 0 ${-table_thickness/2}" />
+      <origin rpy="0 0 0" xyz="0 0 ${table_height -table_thickness/2}" />
       <geometry>
         <box size="${table_length} ${table_width} ${table_thickness}" />

Commit message: maybe

File: Step2/table_macro.xacro (robot description, xacro)
@@ -10,13 +10,13 @@
     <xacro:property name="leg_radius" value="0.05" /> <!-- radius of leg -->
   <!-- joint from "world" to "top"-->
-  <joint name="table_base_joint" type="fixed">
-    <origin rpy="0 0 0" xyz="0 0 0" />
+  <joint name="{prefix}}base_joint" type="fixed">
+    <origin rpy="0 0 0" xyz="0 0 ${table_height}" />
     <parent link="${parent}" />
     <child link="table_top" />
   </joint>
   <!-- Top Link -->
-  <link name="table_top">
+  <link name="{prefix}top">
     <visual>
-      <origin rpy="0 0 0" xyz="0 0 ${table_height -table_thickness/2}" />
+      <origin rpy="0 0 0" xyz="0 0 ${-table_thickness/2}" />
       <geometry>
         <box size="${table_length} ${table_width} ${table_thickness}" />

Commit message: d

File: Step2/table_macro.xacro (robot description, xacro)
@@ -10,8 +10,8 @@
     <xacro:property name="leg_radius" value="0.05" /> <!-- radius of leg -->
   <!-- joint from "world" to "top"-->
-  <joint name="{prefix}}base_joint" type="fixed">
+  <joint name="{prefix}base_joint" type="fixed">
     <origin rpy="0 0 0" xyz="0 0 ${table_height}" />
     <parent link="${parent}" />
-    <child link="table_top" />
+    <child link="{prefix}top" />
   </joint>
   <!-- Top Link -->

Commit message: s

File: Step2/table_macro.xacro (robot description, xacro)
@@ -28,5 +28,5 @@
   <joint name="${prefix}leg1_joint" type="fixed">
     <origin rpy="0 0 0" xyz="${(table_length /2) - leg_radius} ${(table_width / 2) - leg_radius} 0" />
-    <parent link="table_top" />
+    <parent link="{prefix}top" />
     <child link="${prefix}leg1" />
   </joint>
@@ -44,5 +44,5 @@
   <joint name="${prefix}leg2_joint" type="fixed">
     <origin rpy="0 0 0" xyz="-${(table_length /2) - leg_radius}  ${(table_width / 2) - leg_radius} 0" />
-    <parent link="table_top" />
+    <parent link="{prefix}top" />
     <child link="${prefix}leg_link_2" />
   </joint>
@@ -60,5 +60,5 @@
   <joint name="${prefix}leg3_joint" type="fixed">
     <origin rpy="0 0 0" xyz="${(table_length / 2) - leg_radius} -${(table_width / 2) - leg_radius} 0" />
-    <parent link="table_top" />
+    <parent link="{prefix}top" />
     <child link="${prefix}leg_link_3" />
   </joint>
@@ -76,5 +76,5 @@
   <joint name="${prefix}leg4_joint" type="fixed">
     <origin rpy="0 0 0" xyz="-${(table_length /2) - leg_radius} -${(table_width / 2) - leg_radius} 0" />
-    <parent link="table_top" />
+    <parent link="{prefix}top" />
     <child link="${prefix}leg_link_4" />
   </joint>

Commit message: k

File: Step2/table_macro.xacro (robot description, xacro)
@@ -11,5 +11,5 @@
   <!-- joint from "world" to "top"-->
   <joint name="{prefix}base_joint" type="fixed">
-    <origin rpy="0 0 0" xyz="0 0 ${table_height}" />
+    <origin rpy="${pi} 0 0" xyz="0 0 ${table_height}" />
     <parent link="${parent}" />
     <child link="{prefix}top" />
@@ -28,5 +28,5 @@
   <joint name="${prefix}leg1_joint" type="fixed">
     <origin rpy="0 0 0" xyz="${(table_length /2) - leg_radius} ${(table_width / 2) - leg_radius} 0" />
-    <parent link="{prefix}top" />
+    <parent link="table_top" />
     <child link="${prefix}leg1" />
   </joint>

File: Step2/table_on_rrbot.urdf.xacro (robot description, xacro)
@@ -9,5 +9,5 @@
     </xacro:rrbot>
     <xacro:table prefix="table_" parent="rrbot_tool0">
-        <origin xyz="0 0 0" rpy="${2 * pi} ${pi} 0" />
+        <origin xyz="0 0 0" rpy="${pi} 0 0" />
     </xacro:table>
 </robot>

Commit message: d

File: Step2/table_macro.xacro (robot description, xacro)
@@ -28,5 +28,5 @@
   <joint name="${prefix}leg1_joint" type="fixed">
     <origin rpy="0 0 0" xyz="${(table_length /2) - leg_radius} ${(table_width / 2) - leg_radius} 0" />
-    <parent link="table_top" />
+    <parent link="{prefix}top" />
     <child link="${prefix}leg1" />
   </joint>

Commit message: ok

File: Step2/table_macro.xacro (robot description, xacro)
@@ -11,5 +11,5 @@
   <!-- joint from "world" to "top"-->
   <joint name="{prefix}base_joint" type="fixed">
-    <origin rpy="${pi} 0 0" xyz="0 0 ${table_height}" />
+    <origin rpy="${pi} 0 0" xyz="0 0 0" />
     <parent link="${parent}" />
     <child link="{prefix}top" />
@@ -18,5 +18,5 @@
   <link name="{prefix}top">
     <visual>
-      <origin rpy="0 0 0" xyz="0 0 ${-table_thickness/2}" />
+      <origin rpy="0 0 0" xyz="0 0 ${table_height-(table_thickness/2)}" />
       <geometry>
         <box size="${table_length} ${table_width} ${table_thickness}" />

Commit message: ok

File: Step2/table_macro.xacro (robot description, xacro)
@@ -18,5 +18,5 @@
   <link name="{prefix}top">
     <visual>
-      <origin rpy="0 0 0" xyz="0 0 ${table_height-(table_thickness/2)}" />
+      <origin rpy="0 0 0" xyz="0 0 ${-table_thickness/2}" />
       <geometry>
         <box size="${table_length} ${table_width} ${table_thickness}" />

Commit message: d

File: Step2/table_macro.xacro (robot description, xacro)
@@ -11,5 +11,5 @@
   <!-- joint from "world" to "top"-->
   <joint name="{prefix}base_joint" type="fixed">
-    <origin rpy="${pi} 0 0" xyz="0 0 0" />
+    <origin rpy="$0 0 0" xyz="0 0 ${table_height}" />
     <parent link="${parent}" />
     <child link="{prefix}top" />

Commit message: ok

File: Step2/table_macro.xacro (robot description, xacro)
@@ -10,5 +10,5 @@
     <xacro:property name="leg_radius" value="0.05" /> <!-- radius of leg -->
   <!-- joint from "world" to "top"-->
-  <joint name="{prefix}base_joint" type="fixed">
+  <joint name="${prefix}base_joint" type="fixed">
     <origin rpy="$0 0 0" xyz="0 0 ${table_height}" />
     <parent link="${parent}" />
@@ -16,5 +16,5 @@
   </joint>
   <!-- Top Link -->
-  <link name="{prefix}top">
+  <link name="${prefix}top">
     <visual>
       <origin rpy="0 0 0" xyz="0 0 ${-table_thickness/2}" />

Commit message: ok maybe

File: Step2/table_macro.xacro (robot description, xacro)
@@ -13,5 +13,5 @@
     <origin rpy="$0 0 0" xyz="0 0 ${table_height}" />
     <parent link="${parent}" />
-    <child link="{prefix}top" />
+    <child link="${prefix}top" />
   </joint>
   <!-- Top Link -->
@@ -28,5 +28,5 @@
   <joint name="${prefix}leg1_joint" type="fixed">
     <origin rpy="0 0 0" xyz="${(table_length /2) - leg_radius} ${(table_width / 2) - leg_radius} 0" />
-    <parent link="{prefix}top" />
+    <parent link="${prefix}top" />
     <child link="${prefix}leg1" />
   </joint>
@@ -44,5 +44,5 @@
   <joint name="${prefix}leg2_joint" type="fixed">
     <origin rpy="0 0 0" xyz="-${(table_length /2) - leg_radius}  ${(table_width / 2) - leg_radius} 0" />
-    <parent link="{prefix}top" />
+    <parent link="${prefix}top" />
     <child link="${prefix}leg_link_2" />
   </joint>
@@ -60,5 +60,5 @@
   <joint name="${prefix}leg3_joint" type="fixed">
     <origin rpy="0 0 0" xyz="${(table_length / 2) - leg_radius} -${(table_width / 2) - leg_radius} 0" />
-    <parent link="{prefix}top" />
+    <parent link="${prefix}top" />
     <child link="${prefix}leg_link_3" />
   </joint>
@@ -76,5 +76,5 @@
   <joint name="${prefix}leg4_joint" type="fixed">
     <origin rpy="0 0 0" xyz="-${(table_length /2) - leg_radius} -${(table_width / 2) - leg_radius} 0" />
-    <parent link="{prefix}top" />
+    <parent link="${prefix}top" />
     <child link="${prefix}leg_link_4" />
   </joint>

Commit message: okok

File: Step2/table_macro.xacro (robot description, xacro)
@@ -11,5 +11,5 @@
   <!-- joint from "world" to "top"-->
   <joint name="${prefix}base_joint" type="fixed">
-    <origin rpy="$0 0 0" xyz="0 0 ${table_height}" />
+    <origin rpy="0 0 0" xyz="0 0 ${table_height}" />
     <parent link="${parent}" />
     <child link="${prefix}top" />

Commit message: ok maybe tho

File: Step2/table_macro.xacro (robot description, xacro)
@@ -11,5 +11,5 @@
   <!-- joint from "world" to "top"-->
   <joint name="${prefix}base_joint" type="fixed">
-    <origin rpy="0 0 0" xyz="0 0 ${table_height}" />
+    <xacro:insert_block name="origin" />
     <parent link="${parent}" />
     <child link="${prefix}top" />
