Commit message: task4

File: Step2/rrbots_on_tables.urdf.xacro (robot description, xacro)
@@ -5,8 +5,20 @@
     <xacro:include filename="rrbot_macro.xacro" />
     <link name="world" />
-    <xacro:table prefix="table_" parent="world">
-        <origin xyz="0 0 1" rpy="0 0 0" />
+    <xacro:table prefix="table1_" parent="world">
+        <origin xyz="5 0 1" rpy="0 0 0" />
     </xacro:table>
-    <xacro:rrbot prefix="rrbot_" parent="table_top">
+    <xacro:rrbot prefix="rrbot1_" parent="table_top">
+        <origin xyz="0 0 0" rpy="0 0 0" />
+    </xacro:rrbot>
+    <xacro:table prefix="table2_" parent="world">
+        <origin xyz="-2 0 1" rpy="0 0 0" />
+    </xacro:table>
+    <xacro:rrbot prefix="rrbot2_" parent="table_top">
+        <origin xyz="0 0 0" rpy="0 0 0" />
+    </xacro:rrbot>
+        <xacro:table prefix="table3_" parent="world">
+        <origin xyz="6 0 1" rpy="0 0 0" />
+    </xacro:table>
+    <xacro:rrbot prefix="rrbot3_" parent="table_top">
         <origin xyz="0 0 0" rpy="0 0 0" />
     </xacro:rrbot>

File: Step2/table_macro.xacro (robot description, xacro)
@@ -3,5 +3,5 @@
   <xacro:macro name="table" params="prefix parent *origin">
     <!-- Constants for robot dimensions -->
-    <xacro:property name="table_length" value="5" /> <!-- base (x) of top -->
+    <xacro:property name="table_length" value="3" /> <!-- base (x) of top -->
     <xacro:property name="table_width" value="2" /> <!-- width (y) of top  -->
     <xacro:property name="table_height" value="1" /> <!-- height (z) of top -->

Commit message: d

File: Step2/rrbots_on_tables.urdf.xacro (robot description, xacro)
@@ -6,5 +6,5 @@
     <link name="world" />
     <xacro:table prefix="table1_" parent="world">
-        <origin xyz="5 0 1" rpy="0 0 0" />
+        <origin xyz="5 0 1" rpy="0 0 ${degrees(180)}" />
     </xacro:table>
     <xacro:rrbot prefix="rrbot1_" parent="table1_top">

Commit message: m

File: Step2/rrbots_on_tables.urdf.xacro (robot description, xacro)
@@ -1,4 +1,4 @@
 <?xml version="1.0" encoding="UTF-8"?>
-<robot xmlns:xacro="http://wiki.ros.org/xacro" name="table">
+<robot xmlns:xacro="http://wiki.ros.org/xacro" name="rrbot">
     <xacro:include filename="materials.xacro" />
     <xacro:include filename="table_macro.xacro" />
@@ -6,5 +6,5 @@
     <link name="world" />
     <xacro:table prefix="table1_" parent="world">
-        <origin xyz="5 0 1" rpy="0 0 ${degrees(180)}" />
+        <origin xyz="0 0 1" rpy="0 0 ${degrees(180)}" />
     </xacro:table>
     <xacro:rrbot prefix="rrbot1_" parent="table1_top">
@@ -12,5 +12,5 @@
     </xacro:rrbot>
     <xacro:table prefix="table2_" parent="world">
-        <origin xyz="-2 0 1" rpy="0 0 0" />
+        <origin xyz="0 0 1" rpy="0 0 0" />
     </xacro:table>
     <xacro:rrbot prefix="rrbot2_" parent="table2_top">
@@ -18,5 +18,5 @@
     </xacro:rrbot>
         <xacro:table prefix="table3_" parent="world">
-        <origin xyz="6 0 1" rpy="0 0 0" />
+        <origin xyz="0 0 1" rpy="0 0 0" />
     </xacro:table>
     <xacro:rrbot prefix="rrbot3_" parent="table3_top">

Commit message: d

File: Step2/rrbots_on_tables.urdf.xacro (robot description, xacro)
@@ -12,5 +12,5 @@
     </xacro:rrbot>
     <xacro:table prefix="table2_" parent="world">
-        <origin xyz="0 0 1" rpy="0 0 0" />
+        <origin xyz="5 0 1" rpy="0 0 0" />
     </xacro:table>
     <xacro:rrbot prefix="rrbot2_" parent="table2_top">
@@ -18,5 +18,5 @@
     </xacro:rrbot>
         <xacro:table prefix="table3_" parent="world">
-        <origin xyz="0 0 1" rpy="0 0 0" />
+        <origin xyz="-2 6 1" rpy="0 0 0" />
     </xacro:table>
     <xacro:rrbot prefix="rrbot3_" parent="table3_top">

Commit message: d

File: Step2/rrbots_on_tables.urdf.xacro (robot description, xacro)
@@ -5,21 +5,13 @@
     <xacro:include filename="rrbot_macro.xacro" />
     <link name="world" />
-    <xacro:table prefix="table1_" parent="world">
-        <origin xyz="0 0 1" rpy="0 0 ${degrees(180)}" />
-    </xacro:table>
-    <xacro:rrbot prefix="rrbot1_" parent="table1_top">
-        <origin xyz="0 0 0" rpy="0 0 0" />
-    </xacro:rrbot>
-    <xacro:table prefix="table2_" parent="world">
-        <origin xyz="5 0 1" rpy="0 0 0" />
-    </xacro:table>
-    <xacro:rrbot prefix="rrbot2_" parent="table2_top">
-        <origin xyz="0 0 0" rpy="0 0 0" />
-    </xacro:rrbot>
-        <xacro:table prefix="table3_" parent="world">
-        <origin xyz="-2 6 1" rpy="0 0 0" />
-    </xacro:table>
-    <xacro:rrbot prefix="rrbot3_" parent="table3_top">
-        <origin xyz="0 0 0" rpy="0 0 0" />
-    </xacro:rrbot>
+  <!-- create the first robot -->
+  <xacro:rrbot prefix="rrbot1_" parent="world">
+    <!-- position robot in the world -->
+    <origin xyz="0 0 0" rpy="0 0 0" />
+  </xacro:rrbot>
+  <!-- create the second robot -->
+  <xacro:rrbot prefix="rrbot2_" parent="world">
+    <!-- position robot in the world -->
+    <origin xyz="3 0 0" rpy="0 0 ${degrees(180)}" />
+  </xacro:rrbot>
 </robot>

Commit message: ok

File: Step2/rrbots_on_tables.urdf.xacro (robot description, xacro)
@@ -5,13 +5,9 @@
     <xacro:include filename="rrbot_macro.xacro" />
     <link name="world" />
-  <!-- create the first robot -->
-  <xacro:rrbot prefix="rrbot1_" parent="world">
-    <!-- position robot in the world -->
-    <origin xyz="0 0 0" rpy="0 0 0" />
-  </xacro:rrbot>
-  <!-- create the second robot -->
-  <xacro:rrbot prefix="rrbot2_" parent="world">
-    <!-- position robot in the world -->
-    <origin xyz="3 0 0" rpy="0 0 ${degrees(180)}" />
-  </xacro:rrbot>
+    <xacro:table prefix="table1_" parent="world">
+        <origin xyz="3 0 1" rpy="0 0 ${degrees(180)}" />
+    </xacro:table>
+    <xacro:table prefix="table2_" parent="world">
+        <origin xyz="3 0 1" rpy="0 0 ${degrees(180)}" />
+    </xacro:table>
 </robot>

Commit message: d

File: Step2/rrbots_on_tables.urdf.xacro (robot description, xacro)
@@ -9,5 +9,5 @@
     </xacro:table>
     <xacro:table prefix="table2_" parent="world">
-        <origin xyz="3 0 1" rpy="0 0 ${degrees(180)}" />
+        <origin xyz="-1 6 1" rpy="0 0 ${degrees(180)}" />
     </xacro:table>
 </robot>

Commit message: d

File: Step2/rrbots_on_tables.urdf.xacro (robot description, xacro)
@@ -8,6 +8,21 @@
         <origin xyz="3 0 1" rpy="0 0 ${degrees(180)}" />
     </xacro:table>
+    <xacro:rrbot prefix="rrbot1_" parent="world">
+        <!-- position robot in the world -->
+        <origin xyz="3 0 1" rpy="0 0 ${degrees(180)}" />
+    </xacro:rrbot>
     <xacro:table prefix="table2_" parent="world">
-        <origin xyz="-1 6 1" rpy="0 0 ${degrees(180)}" />
+        <origin xyz="-1 6 1" rpy="0 0 0" />
     </xacro:table>
+    <xacro:rrbot prefix="rrbot2_" parent="world">
+        <!-- position robot in the world -->
+        <origin xyz="-1 6 1" rpy="0 0 0" />
+    </xacro:rrbot>
+    <xacro:table prefix="table3_" parent="world">
+        <origin xyz="2 -2 1" rpy="0 0 ${degrees(180)}" />
+    </xacro:table>
+    <xacro:rrbot prefix="rrbot3_" parent="world">
+        <!-- position robot in the world -->
+        <origin xyz="2 -2 1" rpy="0 0 ${degrees(180)}" />
+    </xacro:rrbot>
 </robot>
